File: V1.0/PCB_Files/Weather_Station.kicad_sch (KiCad schematic)
At the start: 36 parts, among them J1 Conn_01x04_Socket, J2 USB_B_Micro, J3 Conn_01x04_Pin, J4 Conn_01x04_Pin, J5 Conn_01x06_Pin, U1 STM32F103C8T6, U2 HDC1080DMBR, U3 AMS1117-3.3, U5 SRV05-4, Y1 X322516MLB4SI

Commit message: Finished first version of routing.
Connections:
- net LED_B: now also U1.2 (PC13); no longer U1.10 (PA0)
- net LED_R: now also U1.3 (PC14); no longer U1.12 (PA2)
- net LED_W: now also U1.4 (PC15); no longer U1.11 (PA1)
- no-connect marks 25 -> 22
Changed lines of the file:
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@@
-	)
-	(no_connect
-		(at 114.3 86.36)
 	)
 	(no_connect
@@
 	)
 	(no_connect
-		(at 114.3 88.9)
-	)
-	(no_connect
 		(at 114.3 119.38)
 	)
@@
 	)
 	(no_connect
-		(at 114.3 83.82)
-	)
-	(no_connect
 		(at 147.32 86.36)
 	)
@@
 	(wire
 		(pts
+			(xy 111.76 88.9) (xy 114.3 88.9)
+		)
+		(stroke
+			(width 0)
+			(type default)
+		)
+	)
+	(wire
+		(pts
 			(xy 88.9 111.76) (xy 114.3 111.76)
 		)
@@
 	(wire
 		(pts
+			(xy 111.76 83.82) (xy 114.3 83.82)
+		)
+		(stroke
+			(width 0)
+			(type default)
+		)
+	)
+	(wire
+		(pts
 			(xy 147.32 91.44) (xy 148.59 91.44)
 		)
@@
 	(wire
 		(pts
+			(xy 175.26 68.58) (xy 190.5 68.58)
+		)
+		(stroke
+			(width 0)
+			(type default)
+		)
+	)
+	(wire
+		(pts
 			(xy 260.35 113.03) (xy 273.05 113.03)
 		)
@@
 		)
 	)
+	(wire
+		(pts
+			(xy 175.26 66.04) (xy 200.66 66.04)
+		)
+		(stroke
+			(width 0)
+			(type default)
+		)
+	)
 	(polyline
 		(pts
@@
 	(wire
 		(pts
+			(xy 111.76 86.36) (xy 114.3 86.36)
+		)
+		(stroke
+			(width 0)
+			(type default)
+		)
+	)
+	(wire
+		(pts
 			(xy 73.66 58.42) (xy 97.79 58.42)
 		)
@@
 	(wire
 		(pts
-			(xy 147.32 66.04) (xy 200.66 66.04)
-		)
-		(stroke
-			(width 0)
-			(type default)
-		)
-	)
-	(wire
-		(pts
 			(xy 289.56 184.15) (xy 289.56 186.69)
 		)
@@
 	(wire
 		(pts
+			(xy 175.26 71.12) (xy 180.34 71.12)
+		)
+		(stroke
+			(width 0)
+			(type default)
+		)
+	)
+	(wire
+		(pts
 			(xy 309.88 186.69) (xy 309.88 185.42)
 		)
@@
 	(wire
 		(pts
-			(xy 147.32 71.12) (xy 180.34 71.12)
-		)
-		(stroke
-			(width 0)
-			(type default)
-		)
-	)
-	(wire
-		(pts
 			(xy 41.91 97.79) (xy 41.91 104.14)
 		)
@@
 		(pts
 			(xy 53.34 213.36) (xy 53.34 218.44)
-		)
-		(stroke
-			(width 0)
-			(type default)
-		)
-	)
-	(wire
-		(pts
-			(xy 147.32 68.58) (xy 190.5 68.58)
 		)
 		(stroke
@@
 		)
 	)
+	(label "LED_B"
+		(at 111.76 83.82 180)
+		(fields_autoplaced yes)
+		(effects
+			(font
+				(size 1.27 1.27)
+			)
+			(justify right bottom)
+		)
+	)
 	(label "I2C1_SDA"
 		(at 261.62 140.97 0)
@@
 		)
 	)
+	(label "LED_R"
+		(at 111.76 86.36 180)
+		(fields_autoplaced yes)
+		(effects
+			(font
+				(size 1.27 1.27)
+			)
+			(justify right bottom)
+		)
+	)
 	(label "USART1_RX"
 		(at 148.59 91.44 0)
@@
 		)
 	)
+	(label "LED_W"
+		(at 111.76 88.9 180)
+		(fields_autoplaced yes)
+		(effects
+			(font
+				(size 1.27 1.27)
+			)
+			(justify right bottom)
+		)
+	)
 	(label "NRST"
 		(at 105.41 66.04 0)
@@
 	)
 	(label "LED_W"
-		(at 148.59 68.58 0)
+		(at 175.26 68.58 0)
 		(fields_autoplaced yes)
 		(effects
@@
 	)
 	(label "LED_R"
-		(at 148.59 71.12 0)
+		(at 175.26 71.12 0)
 		(fields_autoplaced yes)
 		(effects
@@
 	)
 	(label "LED_B"
-		(at 148.59 66.04 0)
-		(fields_autoplaced yes)
-		(effects
+		(at 175.26 66.04 0)
+		(fields_autoplaced yes)
+		(effects

Commit message: Changed Micro USB to USB.
Parts:
- removed J2: USB_B_Micro, Connector_USB:USB_Mini-B_Lumberg_2486_01_Horizontal, symbol Connector:USB_B_Micro
- added J2: TYPE-C16PIN, Connector_USB:USB_C_Receptacle_GCT_USB4105-xx-A_16P_TopMnt_Horizontal, symbol Connector:USB_C_Receptacle_USB2.0_14P
- added R4: 5k1, Resistor_SMD:R_0603_1608Metric, symbol Device:R
- added R9: 1M, Resistor_SMD:R_0603_1608Metric, symbol Device:R
- R5: value 1k5 -> 5k1
Connections:
- net GND: now also R5.2, J2.A1 (GND), J2.A12 (GND), J2.B1 (GND), J2.B12 (GND), R4.1, R9.1
- net USB_D+: now also U5.3 (IO2), U5.4 (IO3), J2.A6 (D+), J2.B6 (D+); no longer R5.2, U5.1 (IO1), U5.6 (IO4)
- net USB_D-: now also U5.1 (IO1), U5.6 (IO4), J2.A7 (D-), J2.B7 (D-); no longer U5.3 (IO2), U5.4 (IO3)
- net VBUS: no longer R5.1
- net VBUS_IN: now also J2.A4 (VBUS), J2.A9 (VBUS), J2.B4 (VBUS), J2.B9 (VBUS)
- new net: J2.S1 (SHIELD), R9.2
- new net CC1: J2.A5 (CC1), R4.2
- new net CC2: J2.B5 (CC2), R5.1
- no-connect marks 22 -> 21
Other:
- moved on the sheet: F1

Commit message: V1.0 should be finished.
Connections:
- net RTC_CLK: now also U1.18 (PB0)
- net RTC_INT: now also U1.19 (PB1)
- no-connect marks 21 -> 26
Changed lines of the file:
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@@
+	)
+	(no_connect
+		(at 146.05 210.82)
 	)
 	(no_connect
@@
 	)
 	(no_connect
+		(at 147.32 66.04)
+	)
+	(no_connect
 		(at 147.32 81.28)
 	)
@@
 	)
 	(no_connect
+		(at 146.05 208.28)
+	)
+	(no_connect
 		(at 114.3 119.38)
 	)
@@
 	)
 	(no_connect
+		(at 147.32 71.12)
+	)
+	(no_connect
 		(at 114.3 127)
 	)
@@
 	)
 	(no_connect
+		(at 147.32 68.58)
+	)
+	(no_connect
+		(at 146.05 205.74)
+	)
+	(no_connect
 		(at 147.32 86.36)
 	)
 	(no_connect
-		(at 114.3 96.52)
-	)
-	(no_connect
-		(at 114.3 93.98)
+		(at 146.05 203.2)
 	)
 	(wire
@@
 	(wire
 		(pts
+			(xy 111.76 93.98) (xy 114.3 93.98)
+		)
+		(stroke
+			(width 0)
+			(type default)
+		)
+	)
+	(wire
+		(pts
 			(xy 58.42 36.83) (xy 76.2 36.83)
 		)
@@
 		(pts
 			(xy 59.69 104.14) (xy 82.55 104.14)
+		)
+		(stroke
+			(width 0)
+			(type default)
+		)
+	)
+	(wire
+		(pts
+			(xy 111.76 96.52) (xy 114.3 96.52)
 		)
 		(stroke
@@
 		)
 	)
+	(label "RTC_CLK"
+		(at 111.76 93.98 180)
+		(fields_autoplaced yes)
+		(effects
+			(font
+				(size 1.27 1.27)
+			)
+			(justify right bottom)
+		)
+	)
 	(label "USART1_RX"
 		(at 260.35 115.57 0)
@@
 		)
 	)
+	(label "RTC_INT"
+		(at 111.76 96.52 180)
+		(fields_autoplaced yes)
+		(effects
+			(font
+				(size 1.27 1.27)
+			)
+			(justify right bottom)
+		)
+	)

Commit message: DRC is to do but otherwise should be V1.
Parts:
- J1: value Conn_01x04_Socket -> HS91L02W2C01
- J3, J4: value Conn_01x04_Pin -> B-2100S04P-A110
- J5: value Conn_01x06_Pin -> ZX-PZ2.54-1-6PZZ
Other:
- note added: "Display"
Changed lines of the file:
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@@
 		)
 	)
+	(polyline
+		(pts
+			(xy 127 193.04) (xy 127 217.17)
+		)
+		(stroke
+			(width 0)
+			(type dash)
+		)
+	)
 	(wire
 		(pts
@@
 		)
 	)
+	(polyline
+		(pts
+			(xy 148.59 217.17) (xy 127 217.17)
+		)
+		(stroke
+			(width 0)
+			(type dash)
+		)
+	)
 	(wire
 		(pts
@@
 		)
 	)
+	(polyline
+		(pts
+			(xy 127 193.04) (xy 148.59 193.04)
+		)
+		(stroke
+			(width 0)
+			(type dash)
+		)
+	)
 	(wire
 		(pts
@@
 		)
 	)
+	(polyline
+		(pts
+			(xy 148.59 193.04) (xy 148.59 217.17)
+		)
+		(stroke
+			(width 0)
+			(type dash)
+		)
+	)
 	(wire
 		(pts
@@
 		)
 	)
+	(text "Display"
+		(exclude_from_sim no)
+		(at 137.16 196.85 0)
+		(effects
+			(font
+				(size 2.54 2.54)
+			)
+		)
+	)
 	(text "Sensor"
 		(exclude_from_sim no)
@@
 			)
 		)
-		(property "Value" "Conn_01x04_Pin"
+		(property "Value" "B-2100S04P-A110"
 			(at 161.29 213.36 0)
 			(effects
@@
 			)
 		)
-		(property "Value" "Conn_01x04_Socket"
+		(property "Value" "HS91L02W2C01"
 			(at 138.43 213.36 0)
 			(effects
@@
 			)
 		)
-		(property "Description" "Generic connector, single row, 01x04, script generated"
+		(property "Description" "Display"
 			(at 140.97 205.74 0)
 			(effects
@@
 			)
 		)
-		(property "Value" "Conn_01x06_Pin"
+		(property "Value" "ZX-PZ2.54-1-6PZZ"
 			(at 279.4 143.5099 0)
 			(effects
@@
 			)
 		)
-		(property "Value" "Conn_01x04_Pin"
+		(property "Value" "B-2100S04P-A110"
 			(at 279.4 118.1101 0)
 			(effects

Commit message: Changed Fuse and added SWD Restistor.
Parts:
- added R10, R11: 100R, Resistor_SMD:R_0603_1608Metric, symbol Device:R
- added R12: 1k5, Resistor_SMD:R_0603_1608Metric, symbol Device:R
- F1: value JFC1206-1100FS -> CFS06V3T1R0; footprint Fuse:Fuse_1206_3216Metric -> Fuse:Fuse_0603_1608Metric
Connections:
- net SWCLK: now also R10.2; no longer U1.37 (PA14)
- net SWDIO: now also R11.2; no longer U1.38 (PA15)
- net USB_D+: now also R12.2
- net VBUS: now also R12.1
- new net uC_SWCLK: R10.1, U1.37 (PA14)
- new net uC_SWDIO: R11.1, U1.38 (PA15)
