File: Solar Module/V1.0/Solar_Module.kicad_pcb (KiCad board)
At the start: 4 copper layers, 34.2 x 19.5 mm, 23 parts, among them J1 B2B-PH-K-S, J2 TYPE-C16PIN, J3 B2B-PH-K-S, U1 MT3608, U2 TP4057

Commit message: Nothing really changed.
Parts:
- added R5: 2k, Resistor_SMD:R_0603_1608Metric, F.Cu at (174.8, 60.0)
- D2: value LED -> KT-0603G
- D3: value LED -> KT-0603R
- L1: value MDA7030-150M -> CYA0630-15UH; footprint Inductor_SMD:L_Sunlord_MWSA0603S -> Inductor_SMD:L_Chilisin_BMRx00060615
- R3: value 4k -> 2k
- turned R8 to 90 degrees
Connections:
- R3 pad 2: GND -> Net-(R3-Pad2)
Routing:
- net Net-(R3-Pad2): track 0.00 -> 1.50 mm
- net GND: vias 30 -> 32
