File: Solar Module/V1.0/Solar_Module.kicad_sch (KiCad schematic)
At the start: 23 parts, among them J1 B2B-PH-K-S, J2 TYPE-C16PIN, J3 B2B-PH-K-S, U1 MT3608, U2 TP4057

Commit message: Added BOMS and added notes in schematic.
Parts:
- L1: value MDA7030-150M -> CYA0630-15UH; footprint Inductor_SMD:L_Sunlord_MWSA0603S -> Inductor_SMD:L_Chilisin_BMRx00060615
Changed lines of the file:
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@@
+		)
+	)
+	(text_box "Change to CYA0630-15UH on PCB"
+		(exclude_from_sim no)
+		(at 54.61 30.48 0)
+		(size 19.05 8.89)
+		(stroke
+			(width 0)
+			(type default)
+		)
+		(fill
+			(type color)
+			(color 0 255 255 1)
+		)
+		(effects
+			(font
+				(size 1.27 1.27)
+			)
+			(justify left top)
+		)
+	)
+	(text_box "Change R3 to 2x 2k in Series."
+		(exclude_from_sim no)
+		(at 217.17 90.17 0)
+		(size 19.05 8.89)
+		(stroke
+			(width 0)
+			(type default)
+		)
+		(fill
+			(type color)
+			(color 0 255 255 1)
+		)
+		(effects
+			(font
+				(size 1.27 1.27)
+			)
+			(justify left top)
 		)
 	)
@@
 			)
 		)
-		(property "Value" "MDA7030-150M"
+		(property "Value" "CYA0630-15UH"
 			(at 63.5 44.45 90)
 			(effects
@@
 			)
 		)
-		(property "Footprint" "Inductor_SMD:L_Sunlord_MWSA0603S"
+		(property "Footprint" "Inductor_SMD:L_Chilisin_BMRx00060615"
 			(at 63.5 46.99 0)
 			(effects

Commit message: Nothing really changed.
Parts:
- added R5: 2k, Resistor_SMD:R_0603_1608Metric, symbol Device:R
- R3: value 4k -> 2k
Connections:
- net GND: now also R5.2; no longer R3.2
- new net: R3.2, R5.1
Other:
- moved on the sheet: J1, R3
